Commit message: Video1_5

File: Video1_4/Mecanum/src/mecanum_description/urdf/mecanum_urdf.urdf (robot description, URDF)
Before this commit: robot mecanum_car, 6 links, 5 joints
Links:
- added link base_footprint
Joints:
- added joint joint_base_footprint: type fixed, parent base_footprint, child base_link, origin xyz=0.0 0.0 0.037 rpy=0.0 0.0 0.0

File: Video1_4/Mecanum/src/mecanum_description/xacro/model/wheel1/wheel1.xacro (robot description, xacro)
@@ -20,5 +20,5 @@
                 <origin xyz="0 0 0" rpy="0 0 0" />
                 <geometry>
-                    <cylinder length="0.1" radius="0.05"/>
+                    <cylinder length="0.028" radius="0.014"/>
                 </geometry>
             </collision>
